File: STM32Dev/STM32Dev.kicad_pcb (KiCad board)
At the start: 2 copper layers, 36.2 x 38.1 mm, 31 parts, among them J1 JTAG, J3 USB_C_Receptacle_USB2.0_14P, J4 RIGHT, J5 LEFT, SW1 RST, SW2 BOOT, U2 NCP1117-3.3_SOT223, U3 TVS1400DRV, U4 STM32F411RCTx, Y1 25MHz

Commit message: added trace
Routing:
- net /PB4: track 0.00 -> 15.6 mm
